File: pcb/sensor/sensor.kicad_sch (KiCad schematic)
At the start: 35 parts, among them J1 Conn_01x05, J2 Conn_01x05, SW1 B, SW10 D, SW11 C#, SW12 C, SW2 A#, SW3 A, SW4 G#, SW5 G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

Commit message: Sensor v0
Parts:
- removed H4: MountingHole, MountingHole:MountingHole_3.2mm_M3, symbol Mechanical:MountingHole
- R13: value 10k -> 100k
- SW1, SW10, SW11, SW12, SW2, SW3, SW4, SW5, SW6, SW7, SW8, SW9: footprint TerminalBlock:TerminalBlock_bornier-3_P5.08mm -> Button_Switch_THT:Mini Limit Switch; symbol Switch:SW_Reed -> Switch:SW_Push_SPDT
Connections:
- net GND: now also SW1.3 (C), SW10.3 (C), SW11.3 (C), SW12.3 (C), SW2.3 (C), SW3.3 (C), SW4.3 (C), SW5.3 (C), SW6.3 (C), SW7.3 (C), SW8.3 (C), SW9.3 (C); no longer SW1.1, SW10.1, SW11.1, SW12.1, SW2.1, SW3.1, SW4.1, SW5.1, SW6.1, SW7.1, SW8.1, SW9.1
- net at SW1.2 (B), U1.11 (D0): no longer R1.2
- net at SW5.2 (B), U1.3 (D4): no longer R5.2
- net at SW11.2 (B), U2.13 (D2): no longer R11.2
- net at SW8.2 (B), U1.6 (D7): no longer R8.2
- net at SW10.2 (B), U2.12 (D1): no longer R10.2
- net at SW9.2 (B), U2.11 (D0): no longer R9.2
- net at SW12.2 (B), U2.14 (D3): no longer R12.2
- net at SW4.2 (B), U1.14 (D3): no longer R4.2
- net at SW2.2 (B), U1.12 (D1): no longer R2.2
- net at SW3.2 (B), U1.13 (D2): no longer R3.2
- net at SW6.2 (B), U1.4 (D5): no longer R6.2
- net at SW7.2 (B), U1.5 (D6): no longer R7.2
- new net: R1.2, SW1.1 (A)
- new net: R5.2, SW5.1 (A)
- new net: R11.2, SW11.1 (A)
- new net: R8.2, SW8.1 (A)
- new net: R10.2, SW10.1 (A)
- new net: R4.2, SW4.1 (A)
- new net: R12.2, SW12.1 (A)
- new net: R2.2, SW2.1 (A)
- new net: R3.2, SW3.1 (A)
- new net: R6.2, SW6.1 (A)
- new net: R7.2, SW7.1 (A)
- new net: R9.2, SW9.1 (A)
Other:
- moved on the sheet: R10, R11, R12, R5, R6, R7, R8, R9

Commit message: Checkpoint
Parts:
- removed R1, R10, R11, R2, R3, R4, R5, R6, R7, R8, R9: 10k, Resistor_THT:R_Axial_DIN0207_L6.3mm_D2.5mm_P10.16mm_Horizontal, symbol Device:R
Connections:
- net GND: now also SW1.1 (A), SW10.1 (A), SW11.1 (A), SW12.1 (A), SW2.1 (A), SW3.1 (A), SW4.1 (A), SW5.1 (A), SW6.1 (A), SW7.1 (A), SW8.1 (A), SW9.1 (A); no longer SW1.3 (C), SW10.3 (C), SW11.3 (C), SW12.3 (C), SW2.3 (C), SW3.3 (C), SW4.3 (C), SW5.3 (C), SW6.3 (C), SW7.3 (C), SW8.3 (C), SW9.3 (C)
- net at R12.2: now also SW1.3 (C), SW10.3 (C), SW11.3 (C), SW12.3 (C), SW2.3 (C), SW3.3 (C), SW4.3 (C), SW5.3 (C), SW6.3 (C), SW7.3 (C), SW8.3 (C), SW9.3 (C); no longer SW12.1 (A)
Other:
- moved on the sheet: SW1, SW10, SW11, SW12, SW2, SW3, SW4, SW5, SW6, SW7, SW8, SW9

Commit message: Boards ordered.
Parts:
- J1: value Conn_01x05 -> In; footprint Connector_PinHeader_2.54mm:PinHeader_1x05_P2.54mm_Vertical -> Connector_PinHeader_2.54mm:PinHeader_1x06_P2.54mm_Vertical; symbol Connector_Generic:Conn_01x05 -> Connector_Generic:Conn_01x06
- J2: value Conn_01x05 -> Out; footprint Connector_PinHeader_2.54mm:PinHeader_1x05_P2.54mm_Vertical -> Connector_PinHeader_2.54mm:PinHeader_1x06_P2.54mm_Vertical; symbol Connector_Generic:Conn_01x05 -> Connector_Generic:Conn_01x06
Connections:
- net GND: now also J1.6 (Pin_6), J2.6 (Pin_6)
Changed lines of the file:
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@@
+    (pin "1")
+  )
+  (symbol (lib_id "power:GND") (at 99.314 44.196 90) (unit 1)
+    (in_bom yes) (on_board yes) (fields_autoplaced)
+    (property "Reference" "#PWR03" (id 0) (at 105.664 44.196 0)
+      (effects (font (size 1.27 1.27)) hide)
+    )
+    (property "Value" "GND" (id 1) (at 103.632 44.1959 90)
+      (effects (font (size 1.27 1.27)) (justify right))
+    )
+    (property "Footprint" "" (id 2) (at 99.314 44.196 0)
+      (effects (font (size 1.27 1.27)) hide)
+    )
+    (property "Datasheet" "" (id 3) (at 99.314 44.196 0)
+      (effects (font (size 1.27 1.27)) hide)
+    )
     (pin "1")
   )
@@
     )
     (property "Datasheet" "" (id 3) (at 107.188 133.858 0)
+      (effects (font (size 1.27 1.27)) hide)
+    )
+    (pin "1")
+  )
+  (symbol (lib_id "power:GND") (at 75.692 29.718 90) (unit 1)
+    (in_bom yes) (on_board yes) (fields_autoplaced)
+    (property "Reference" "#PWR01" (id 0) (at 82.042 29.718 0)
+      (effects (font (size 1.27 1.27)) hide)
+    )
+    (property "Value" "GND" (id 1) (at 80.01 29.7179 90)
+      (effects (font (size 1.27 1.27)) (justify right))
+    )
+    (property "Footprint" "" (id 2) (at 75.692 29.718 0)
+      (effects (font (size 1.27 1.27)) hide)
+    )
+    (property "Datasheet" "" (id 3) (at 75.692 29.718 0)
       (effects (font (size 1.27 1.27)) hide)
     )
@@
     (pin "3")
   )
-  (symbol (lib_id "Connector_Generic:Conn_01x05") (at 94.234 36.576 0) (mirror y) (unit 1)
+  (symbol (lib_id "Connector_Generic:Conn_01x06") (at 94.234 36.576 0) (mirror y) (unit 1)
     (in_bom yes) (on_board yes) (fields_autoplaced)
     (property "Reference" "J2" (id 0) (at 94.234 25.4 0))
-    (property "Value" "Conn_01x05" (id 1) (at 94.234 27.94 0))
-    (property "Footprint" "Connector_PinHeader_2.54mm:PinHeader_1x05_P2.54mm_Vertical" (id 2) (at 94.234 36.576 0)
+    (property "Value" "Out" (id 1) (at 94.234 27.94 0))
+    (property "Footprint" "Connector_PinHeader_2.54mm:PinHeader_1x06_P2.54mm_Vertical" (id 2) (at 94.234 36.576 0)
       (effects (font (size 1.27 1.27)) hide)
     )
@@
     (pin "4")
     (pin "5")
-  )
-  (symbol (lib_id "Connector_Generic:Conn_01x05") (at 70.612 37.338 180) (unit 1)
-    (in_bom yes) (on_board yes) (fields_autoplaced)
+    (pin "6")
+  )
+  (symbol (lib_id "Connector_Generic:Conn_01x06") (at 70.612 37.338 180) (unit 1)
+    (in_bom yes) (on_board yes)
     (property "Reference" "J1" (id 0) (at 70.612 25.4 0))
-    (property "Value" "Conn_01x05" (id 1) (at 70.612 27.94 0))
-    (property "Footprint" "Connector_PinHeader_2.54mm:PinHeader_1x05_P2.54mm_Vertical" (id 2) (at 70.612 37.338 0)
+    (property "Value" "In" (id 1) (at 70.612 27.178 0))
+    (property "Footprint" "Connector_PinHeader_2.54mm:PinHeader_1x06_P2.54mm_Vertical" (id 2) (at 70.612 37.338 0)
       (effects (font (size 1.27 1.27)) hide)
     )
@@
     (pin "4")
     (pin "5")
+    (pin "6")
   )
   (symbol (lib_id "Switch:SW_Push_SPDT") (at 181.102 130.302 90) (mirror x) (unit 1)
@@
       (reference "#FLG02") (unit 1) (value "PWR_FLAG") (footprint "")
     )
+    (path "/82be7226-1774-4399-a7bf-4684a49bd0ec"
+      (reference "#PWR01") (unit 1) (value "GND") (footprint "")
+    )
     (path "/14ca477a-1b41-4b30-9c5c-6d935d067113"
       (reference "#PWR02") (unit 1) (value "GND") (footprint "")
     )
+    (path "/7bba2cb3-7cc7-4dd3-bb4c-4b61d4bd219c"
+      (reference "#PWR03") (unit 1) (value "GND") (footprint "")
+    )
     (path "/faa016cf-d873-4761-9c13-50706be8eb97"
       (reference "#PWR04") (unit 1) (value "GND") (footprint "")
@@
     )
     (path "/c3d3f615-f1c1-4e64-afca-e8ce55fc4568"
-      (reference "J1") (unit 1) (value "Conn_01x05") (footprint "Connector_PinHeader_2.54mm:PinHeader_1x05_P2.54mm_Vertical")
+      (reference "J1") (unit 1) (value "In") (footprint "Connector_PinHeader_2.54mm:PinHeader_1x06_P2.54mm_Vertical")
     )
     (path "/c287ab95-9c9a-4b76-966a-a3eca1e81f82"
-      (reference "J2") (unit 1) (value "Conn_01x05") (footprint "Connector_PinHeader_2.54mm:PinHeader_1x05_P2.54mm_Vertical")
+      (reference "J2") (unit 1) (value "Out") (footprint "Connector_PinHeader_2.54mm:PinHeader_1x06_P2.54mm_Vertical")
     )
     (path "/3b8c8776-f869-48c3-b437-62b86c285104"
