File: pcb/sensor/sensor.kicad_pcb (KiCad board)
At the start: 2 copper layers, 163.2 x 35 mm, 35 parts, among them J1 Conn_01x05, J2 Conn_01x05, SW1 B, SW10 D, SW11 C#, SW12 C, SW2 A#, SW3 A, SW4 G#, SW5 G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

Commit message: Sensor v0
Parts:
- removed H4: MountingHole, MountingHole:MountingHole_3.2mm_M3
- R13: value 10k -> 100k
- SW1, SW10, SW11, SW12, SW2, SW3, SW4, SW5, SW6, SW7, SW8, SW9: footprint TerminalBlock:TerminalBlock_bornier-3_P5.08mm -> Button_Switch_THT:Mini Limit Switch
- moved H3 77.8 mm to (145.4, 86.1)
- moved U1 12.2 mm to (177.8, 95.6)
- moved C2 12.2 mm to (174.4, 88.0)
- moved J1 12.2 mm to (222.5, 97.6)
- moved J2 11.9 mm to (68.2, 97.7)
- moved C1 11.7 mm to (92.6, 87.8)
- moved U2 11.7 mm to (96.1, 95.5)
- moved R7 8.67 mm to (131.7, 112.7)
- moved R12 8.25 mm to (87.8, 89.6), turned to 180 degrees
- moved SW7 7.84 mm to (138.5, 112.7)
- moved R6 6.82 mm to (145.5, 112.7)
- moved R13 6.31 mm to (215.3, 94.8)
- moved SW6 5.89 mm to (152.4, 112.7)
- moved SW12 5.45 mm to (70.4, 112.7)
- moved R5 5.37 mm to (158.9, 112.7)
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Connections:
- R1 pad 2: Net-(R1-Pad2) -> Net-(SW1-Pad1)
- R11 pad 2: Net-(R11-Pad2) -> Net-(SW11-Pad1)
- R12 pad 2: Net-(R12-Pad2) -> Net-(SW12-Pad1)
- R5 pad 2: Net-(R5-Pad2) -> Net-(SW5-Pad1)
- R6 pad 2: Net-(R6-Pad2) -> Net-(SW6-Pad1)
- R8 pad 2: Net-(R8-Pad2) -> Net-(SW8-Pad1)
- SW1 pad 1: GND -> Net-(SW1-Pad1)
- SW1 pad 2: Net-(R1-Pad2) -> Net-(U1-Pad11)
- SW1 pad 3: (no net) -> GND
- SW10 pad 1: GND -> Net-(R10-Pad2)
- SW10 pad 2: Net-(R10-Pad2) -> Net-(U2-Pad12)
- SW10 pad 3: (no net) -> GND
- SW11 pad 1: GND -> Net-(SW11-Pad1)
- SW11 pad 2: Net-(R11-Pad2) -> Net-(U2-Pad13)
- SW11 pad 3: (no net) -> GND
- SW12 pad 1: GND -> Net-(SW12-Pad1)
- SW12 pad 2: Net-(R12-Pad2) -> Net-(U2-Pad14)
- SW12 pad 3: (no net) -> GND
- SW2 pad 1: GND -> Net-(R2-Pad2)
- SW2 pad 2: Net-(R2-Pad2) -> Net-(U1-Pad12)
- SW2 pad 3: (no net) -> GND
- SW3 pad 1: GND -> Net-(R3-Pad2)
- SW3 pad 2: Net-(R3-Pad2) -> Net-(U1-Pad13)
- SW3 pad 3: (no net) -> GND
- SW4 pad 1: GND -> Net-(R4-Pad2)
- SW4 pad 2: Net-(R4-Pad2) -> Net-(U1-Pad14)
- SW4 pad 3: (no net) -> GND
- SW5 pad 1: GND -> Net-(SW5-Pad1)
- SW5 pad 2: Net-(R5-Pad2) -> Net-(U1-Pad3)
- SW5 pad 3: (no net) -> GND
- SW6 pad 1: GND -> Net-(SW6-Pad1)
- SW6 pad 2: Net-(R6-Pad2) -> Net-(U1-Pad4)
- SW6 pad 3: (no net) -> GND
- SW7 pad 1: GND -> Net-(R7-Pad2)
- SW7 pad 2: Net-(R7-Pad2) -> Net-(U1-Pad5)
- SW7 pad 3: (no net) -> GND
- SW8 pad 1: GND -> Net-(SW8-Pad1)
- SW8 pad 2: Net-(R8-Pad2) -> Net-(U1-Pad6)
- SW8 pad 3: (no net) -> GND
- SW9 pad 1: GND -> Net-(R9-Pad2)
- SW9 pad 2: Net-(R9-Pad2) -> Net-(U2-Pad11)
- SW9 pad 3: (no net) -> GND
- U1 pad 11: Net-(R1-Pad2) -> Net-(U1-Pad11)
- U1 pad 12: Net-(R2-Pad2) -> Net-(U1-Pad12)
- U1 pad 13: Net-(R3-Pad2) -> Net-(U1-Pad13)
- U1 pad 14: Net-(R4-Pad2) -> Net-(U1-Pad14)
- U1 pad 3: Net-(R5-Pad2) -> Net-(U1-Pad3)
- U1 pad 4: Net-(R6-Pad2) -> Net-(U1-Pad4)
- U1 pad 5: Net-(R7-Pad2) -> Net-(U1-Pad5)
- U1 pad 6: Net-(R8-Pad2) -> Net-(U1-Pad6)
- U2 pad 11: Net-(R9-Pad2) -> Net-(U2-Pad11)
- U2 pad 12: Net-(R10-Pad2) -> Net-(U2-Pad12)
- U2 pad 13: Net-(R11-Pad2) -> Net-(U2-Pad13)
- U2 pad 14: Net-(R12-Pad2) -> Net-(U2-Pad14)
Routing:
- net GND: track 327.5 -> 231.2 mm
- net Net-(U1-Pad6): track 0.00 -> 81.3 mm
- net Net-(R8-Pad2): track 71.5 -> 0.00 mm
- net Net-(U1-Pad5): track 0.00 -> 64.8 mm
- net Net-(R12-Pad2): track 48.7 -> 0.00 mm
- net Net-(U1-Pad4): track 0.00 -> 47.7 mm
- net Net-(R11-Pad2): track 47.1 -> 0.00 mm
- net Net-(U2-Pad14): track 0.00 -> 46.0 mm
- net Net-(R1-Pad2): track 45.4 -> 0.00 mm
- net Net-(R7-Pad2): track 48.4 -> 6.81 mm
- net Net-(U1-Pad11): track 0.00 -> 40.3 mm
- net Net-(U2-Pad13): track 0.00 -> 37.9 mm
- net Net-(U2-Pad12): track 0.00 -> 36.1 mm
- net Net-(U1-Pad12): track 0.00 -> 35.8 mm
- net Net-(R6-Pad2): track 33.5 -> 0.00 mm
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Other:
- board size 163.2 x 35 mm -> 162.1 x 40 mm
- board text added: "<"
- board text added: "MK Sensor v0 - 2023-01-08 - joewing.net"
- board text removed: "3DPMK Sensor v0 - 2023-01-08 - joewing.net"
- board text removed: "<<"

Commit message: Checkpoint
Parts:
- removed R1, R10, R11, R2, R3, R4, R5, R6, R7, R8, R9: 10k, Resistor_THT:R_Axial_DIN0207_L6.3mm_D2.5mm_P10.16mm_Horizontal
- moved R12 13.4 mm to (76.8, 97.3), turned to -90 degrees
- moved SW8 10.3 mm to (124.4, 102.4), turned to -90 degrees
- moved SW7 10.3 mm to (138.4, 102.4), turned to -90 degrees
- moved SW9 10.3 mm to (111.4, 102.4), turned to -90 degrees
- moved SW1 10.3 mm to (220.4, 102.4), turned to -90 degrees
- moved SW10 10.3 mm to (97.4, 102.5), turned to -90 degrees
- moved SW11 10.3 mm to (83.4, 102.4), turned to -90 degrees
- moved SW12 10.3 mm to (70.4, 102.4), turned to -90 degrees
- moved SW2 10.3 mm to (206.4, 102.4), turned to -90 degrees
- moved SW4 10.3 mm to (179.4, 102.4), turned to -90 degrees
- moved SW5 10.3 mm to (165.4, 102.4), turned to -90 degrees
- moved SW6 10.3 mm to (152.4, 102.4), turned to -90 degrees
- moved SW3 10.2 mm to (193.4, 102.5), turned to -90 degrees
Connections:
- R12 pad 2: Net-(SW12-Pad1) -> Net-(SW7-Pad3)
- SW1 pad 1: Net-(SW1-Pad1) -> GND
- SW1 pad 3: GND -> Net-(SW7-Pad3)
- SW10 pad 1: Net-(R10-Pad2) -> GND
- SW10 pad 3: GND -> Net-(SW7-Pad3)
- SW11 pad 1: Net-(SW11-Pad1) -> GND
- SW11 pad 3: GND -> Net-(SW7-Pad3)
- SW12 pad 1: Net-(SW12-Pad1) -> GND
- SW12 pad 3: GND -> Net-(SW7-Pad3)
- SW2 pad 1: Net-(R2-Pad2) -> GND
- SW2 pad 3: GND -> Net-(SW7-Pad3)
- SW3 pad 1: Net-(R3-Pad2) -> GND
- SW3 pad 3: GND -> Net-(SW7-Pad3)
- SW4 pad 1: Net-(R4-Pad2) -> GND
- SW4 pad 3: GND -> Net-(SW7-Pad3)
- SW5 pad 1: Net-(SW5-Pad1) -> GND
- SW5 pad 3: GND -> Net-(SW7-Pad3)
- SW6 pad 1: Net-(SW6-Pad1) -> GND
- SW6 pad 3: GND -> Net-(SW7-Pad3)
- SW7 pad 1: Net-(R7-Pad2) -> GND
- SW7 pad 3: GND -> Net-(SW7-Pad3)
- SW8 pad 1: Net-(SW8-Pad1) -> GND
- SW8 pad 3: GND -> Net-(SW7-Pad3)
- SW9 pad 1: Net-(R9-Pad2) -> GND
- SW9 pad 3: GND -> Net-(SW7-Pad3)
Routing:
- net Net-(SW7-Pad3): track 0.00 -> 150.2 mm
- net VCC: track 302.3 -> 258.8 mm
- net GND: track 231.2 -> 268.8 mm
- net Net-(SW12-Pad1): track 15.9 -> 0.00 mm
- net Net-(SW9-Pad2): track 27.4 -> 15.6 mm
- net Net-(SW11-Pad2): track 37.9 -> 27.6 mm
- net Net-(SW2-Pad2): track 35.8 -> 25.5 mm
- net Net-(SW3-Pad2): track 28.1 -> 17.9 mm
- net Net-(SW4-Pad2): track 27.1 -> 17.3 mm, vias 1 -> 0
- net Net-(SW7-Pad2): track 64.8 -> 55.0 mm
- net Net-(SW10-Pad2): track 36.1 -> 26.5 mm
- net Net-(SW6-Pad2): track 47.7 -> 38.1 mm
- net Net-(SW8-Pad2): track 81.3 -> 72.0 mm
- net Net-(SW5-Pad2): track 31.1 -> 21.9 mm
- net Net-(SW12-Pad2): track 46.0 -> 36.8 mm
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Other:
- board text added: "MK Sensor v1 - 2023-01-14 - joewing.net"
- board text removed: "MK Sensor v0 - 2023-01-08 - joewing.net"

Commit message: Boards ordered.
Parts:
- J1: value Conn_01x05 -> In; footprint Connector_PinHeader_2.54mm:PinHeader_1x05_P2.54mm_Vertical -> Connector_PinHeader_2.54mm:PinHeader_1x06_P2.54mm_Vertical; moved to F.Cu
- J2: value Conn_01x05 -> Out; footprint Connector_PinHeader_2.54mm:PinHeader_1x05_P2.54mm_Vertical -> Connector_PinHeader_2.54mm:PinHeader_1x06_P2.54mm_Vertical
- moved SW8 2.00 mm to (126.4, 102.4)
- moved J2 1.05 mm to (69.2, 98.0)
- moved SW10 1.00 mm to (98.4, 102.5)
- moved SW11 1.00 mm to (84.4, 102.4)
- moved SW2 1.00 mm to (207.4, 102.4)
- moved SW4 1.00 mm to (180.4, 102.4)
- moved SW5 1.00 mm to (166.4, 102.4)
- moved SW6 1.00 mm to (153.4, 102.4)
- moved SW7 1.00 mm to (139.4, 102.4)
- moved SW9 1.00 mm to (112.4, 102.4)
- moved J1 0.98 mm to (221.6, 98.0), turned to 180 degrees
Routing:
- net GND: track 268.8 -> 288.4 mm
- net Net-(SW8-Pad2): track 72.0 -> 70.0 mm
- net SHIFT: track 184.5 -> 182.9 mm
- net ~{LOAD}: track 183.9 -> 182.3 mm
- net IN: track 33.2 -> 32.2 mm
- net Net-(SW7-Pad2): track 55.0 -> 54.0 mm
- net Net-(SW10-Pad2): track 26.5 -> 27.5 mm
- net Net-(SW5-Pad2): track 21.9 -> 20.9 mm
- net Net-(SW4-Pad2): track 17.3 -> 16.4 mm
- net OUT: track 49.0 -> 48.2 mm
- net VCC: track 258.8 -> 258.2 mm
- net Net-(SW6-Pad2): track 38.1 -> 37.5 mm
Other:
- board text added: "MK Sensor v1 - 2023-01-21 - joewing.net"
- board text removed: "MK Sensor v1 - 2023-01-14 - joewing.net"

Commit message: Checkpoint
Parts:
- moved J1 1.00 mm to (220.6, 98.0)
- moved J2 1.00 mm to (70.2, 98.0)
- moved H3 0.10 mm to (145.4, 86.2)
Routing:
- net GND: track 288.4 -> 282.9 mm
- net ~{LOAD}: track 182.3 -> 180.3 mm
- net SHIFT: track 182.9 -> 180.9 mm
- net IN: track 32.2 -> 31.1 mm
- net OUT: track 48.2 -> 47.2 mm
Other:
- board size 162.1 x 40 mm -> 162 x 40 mm
- board text added: "MK Sensor v2 - 2023-02-02 - joewing.net"
- board text removed: "MK Sensor v1 - 2023-01-21 - joewing.net"

Commit message: Boards ordered.
Parts:
- moved J2 0.20 mm to (70.4, 98.0)
- moved J1 0.20 mm to (220.4, 98.0)
Other:
- board text added: "MK Sensor v2 - 2023-02-05 - joewing.net"
- board text removed: "MK Sensor v2 - 2023-02-02 - joewing.net"
Changed lines of the file:
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@@
   )
   (footprint "Connector_PinHeader_2.54mm:PinHeader_1x06_P2.54mm_Vertical" (layer "F.Cu")
-    (at 70.2 98 180)
+    (at 70.4 98 180)
     (descr "Through hole straight pin header, 1x06, 2.54mm pitch, single row")
     (tags "Through hole pin header THT 1x06 2.54mm single row")
@@
   )
   (footprint "Connector_PinHeader_2.54mm:PinHeader_1x06_P2.54mm_Vertical" (layer "F.Cu")
-    (at 220.6 98 180)
+    (at 220.4 98 180)
     (descr "Through hole straight pin header, 1x06, 2.54mm pitch, single row")
     (tags "Through hole pin header THT 1x06 2.54mm single row")
@@
     (effects (font (size 1 1) (thickness 0.15)))
   )
-  (gr_text "MK Sensor v2 - 2023-02-02 - joewing.net" (at 91.9 120.5) (layer "F.SilkS")
-    (effects (font (size 1 1) (thickness 0.15)))
-  )
+  (gr_text "MK Sensor v2 - 2023-02-05 - joewing.net" (at 91.9 120.5) (layer "F.SilkS")
+    (effects (font (size 1 1) (thickness 0.15)))
+  )
