File: pcb/controller/controller.kicad_pcb (KiCad board)
At the start: 2 copper layers, 32 x 100 mm, 17 parts, among them J1 USB_B, J2 ISP, J3 AudioJack3, J4 Conn_01x05, SW1 Function, SW2 Power, U1 ATtiny85-20P

Commit message: Checkpoint
Parts:
- added C3: 0.1u, Capacitor_THT:C_Disc_D3.4mm_W2.1mm_P2.50mm, F.Cu at (129.4, 84.7)
- added R2: 1k, Resistor_THT:R_Axial_DIN0207_L6.3mm_D2.5mm_P10.16mm_Horizontal, F.Cu at (129.4, 71.9)
- J4: footprint Connector_PinHeader_2.54mm:PinHeader_1x05_P2.54mm_Horizontal -> Connector_PinHeader_2.54mm:PinHeader_1x05_P2.54mm_Vertical
- U1: value ATtiny85-20P -> ATtiny85
- moved D1 4.70 mm to (116.1, 86.3), turned to 0 degrees
- moved C4 1.71 mm to (120.4, 71.5)
- moved R1 1.30 mm to (124.6, 72.0)
- moved RV1 1.30 mm to (115.2, 108.2)
- moved SW2 0.61 mm to (117.7, 92.8)
- moved J4 0.32 mm to (131.9, 52.5)
Connections:
- RV1 pad 3: Net-(RV1-Pad3) -> Net-(C3-Pad1)
- U1 pad 3: Net-(RV1-Pad3) -> Net-(R2-Pad1)
Routing:
- net Net-(RV1-Pad3): track 54.5 -> 0.00 mm
- net GND: track 159.2 -> 193.6 mm
- net Net-(C3-Pad1): track 0.00 -> 32.2 mm
- net Net-(R2-Pad1): track 0.00 -> 13.2 mm
- net AUDIO_OUT: track 15.8 -> 22.0 mm
- net Net-(D1-Pad2): track 9.34 -> 7.66 mm
- net SCK: track 91.8 -> 93.4 mm
- net Net-(J1-Pad1): track 59.8 -> 61.1 mm
Other:
- board text added: "MK Controller v1 - 2022-01-14 - joewing.net"
- board text removed: "3DPO Controller v1 - 2022-01-07 - joewing.net"

Commit message: Boards ordered.
Parts:
- J4: value Conn_01x05 -> Keys; footprint Connector_PinHeader_2.54mm:PinHeader_1x05_P2.54mm_Vertical -> Connector_PinHeader_2.54mm:PinHeader_1x06_P2.54mm_Vertical; moved to F.Cu
- moved R1 25.2 mm to (125.9, 97.2), turned to 180 degrees
- moved R2 19.4 mm to (125.9, 91.0), turned to 180 degrees
- moved C3 18.1 mm to (112.5, 91.0), turned to 180 degrees
- moved SW2 12.8 mm to (111.3, 103.9)
- moved D1 12.5 mm to (109.9, 97.2)
- moved C1 9.87 mm to (122.8, 42.7), turned to 90 degrees
- moved C4 7.90 mm to (120.2, 79.4)
- moved C2 6.98 mm to (119.0, 72.7), turned to 0 degrees
- moved U1 5.38 mm to (126.6, 69.5)
- moved RV1 4.94 mm to (119.8, 106.4)
- moved J2 4.46 mm to (107.5, 60.7)
- moved J3 3.10 mm to (106.2, 79.6)
- moved J4 3.02 mm to (128.9, 52.9), turned to 180 degrees
- moved J1 1.38 mm to (117.3, 47.5), turned to 180 degrees
- moved H1 0.14 mm to (105.1, 34.1)
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Routing:
- net VCC: track 77.2 -> 98.1 mm
- net Net-(R2-Pad1): track 13.2 -> 29.1 mm
- net Net-(C3-Pad1): track 32.2 -> 22.5 mm
- net SCK: track 93.4 -> 84.3 mm
- net Net-(J1-Pad1): track 61.1 -> 68.9 mm
- net AUDIO_OUT: track 22.0 -> 17.2 mm
- net Net-(D1-Pad2): track 7.66 -> 3.25 mm
- net GND: track 193.6 -> 197.8 mm, vias 0 -> 1
- net ~{RESET}: track 25.1 -> 21.7 mm
- net Net-(C4-Pad1): track 41.3 -> 38.2 mm
- net MOSI: track 32.3 -> 30.2 mm, vias 1 -> 0
- net DATA: track 20.2 -> 21.8 mm
- net MISO: track 41.5 -> 42.2 mm
Other:
- outline, holes or cut-outs redrawn
- board text added: "<"
- board text added: "MK Controller v1 - 2022-01-21 - joewing.net"
- board text removed: "<<"
- board text removed: "MK Controller v1 - 2022-01-14 - joewing.net"

Commit message: Checkpoint
Parts:
- removed SW1: Function, Button_Switch_THT:SW_PUSH_6mm
- removed SW2: Power, Connector_PinHeader_2.54mm:PinHeader_1x03_P2.54mm_Vertical
- removed U1: ATtiny85, Package_DIP:DIP-8_W7.62mm
- added C10: 0.1u, Capacitor_THT:C_Disc_D3.0mm_W2.0mm_P2.50mm, F.Cu at (130.9, 88.3)
- added C11: 0.1u, Capacitor_THT:C_Disc_D3.0mm_W2.0mm_P2.50mm, F.Cu at (144.9, 88.3)
- added C12: 0.1u, Capacitor_THT:C_Disc_D3.0mm_W2.0mm_P2.50mm, F.Cu at (161.1, 88.2)
- added C13: 0.1u, Capacitor_THT:C_Disc_D3.0mm_W2.0mm_P2.50mm, F.Cu at (174.8, 88.3)
- added C14: 0.1u, Capacitor_THT:C_Disc_D3.0mm_W2.0mm_P2.50mm, F.Cu at (188.9, 88.3)
- added C15: 0.1u, Capacitor_THT:C_Disc_D3.0mm_W2.0mm_P2.50mm, F.Cu at (192.5, 88.3)
- added C5: 0.1u, Capacitor_THT:C_Disc_D3.0mm_W2.0mm_P2.50mm, F.Cu at (159.2, 67.2)
- added C6: 0.1u, Capacitor_THT:C_Disc_D3.0mm_W2.0mm_P2.50mm, F.Cu at (73.0, 88.4)
- added C7: 0.1u, Capacitor_THT:C_Disc_D3.0mm_W2.0mm_P2.50mm, F.Cu at (87.0, 88.2)
- added C8: 0.1u, Capacitor_THT:C_Disc_D3.0mm_W2.0mm_P2.50mm, F.Cu at (102.8, 88.3)
- added C9: 0.1u, Capacitor_THT:C_Disc_D3.0mm_W2.0mm_P2.50mm, F.Cu at (117.0, 88.2)
- added RV10: 2', Potentiometer_THT:Potentiometer_Bourns_PTA3043_Single_Slide, F.Cu at (148.4, 91.7)
- added RV2: 16', Potentiometer_THT:Potentiometer_Bourns_PTA3043_Single_Slide, F.Cu at (76.5, 91.7)
- added RV3: 1 3/5', Potentiometer_THT:Potentiometer_Bourns_PTA3043_Single_Slide, F.Cu at (164.6, 91.6)
- added RV4: 5 1/3', Potentiometer_THT:Potentiometer_Bourns_PTA3043_Single_Slide, F.Cu at (90.4, 91.7)
- added RV5: 1 1/3', Potentiometer_THT:Potentiometer_Bourns_PTA3043_Single_Slide, F.Cu at (178.4, 91.6)
- added RV6: 8', Potentiometer_THT:Potentiometer_Bourns_PTA3043_Single_Slide, F.Cu at (106.4, 91.7)
- added RV7: 1', Potentiometer_THT:Potentiometer_Bourns_PTA3043_Single_Slide, F.Cu at (192.4, 91.6)
- added RV8: 4', Potentiometer_THT:Potentiometer_Bourns_PTA3043_Single_Slide, F.Cu at (120.5, 91.7)
- added RV9: 2 2/3', Potentiometer_THT:Potentiometer_Bourns_PTA3043_Single_Slide, F.Cu at (134.4, 91.7)
- added SW17: Function, Button_Switch_THT:SW_PUSH_6mm, F.Cu at (179.1, 72.5)
- added U2: ATtiny861A, Package_DIP:DIP-20_W7.62mm, F.Cu at (146.5, 77.7)
- C1: footprint Capacitor_THT:CP_Radial_D5.0mm_P2.50mm -> Capacitor_THT:CP_Radial_D5.0mm_P2.00mm
- C2, C3: footprint Capacitor_THT:C_Disc_D3.4mm_W2.1mm_P2.50mm -> Capacitor_THT:C_Disc_D3.0mm_W2.0mm_P2.50mm
- C4: value 10u -> 47u; footprint Capacitor_THT:CP_Radial_D5.0mm_P2.50mm -> Capacitor_THT:CP_Radial_D5.0mm_P2.00mm
- R1, R2: footprint Resistor_THT:R_Axial_DIN0207_L6.3mm_D2.5mm_P10.16mm_Horizontal -> Resistor_THT:R_Axial_DIN0309_L9.0mm_D3.2mm_P15.24mm_Horizontal
- RV1: value 10k -> Volume; footprint Potentiometer_THT:Potentiometer_Bourns_3386P_Vertical -> Potentiometer_THT:Potentiometer_Bourns_PTA3043_Single_Slide
- moved H2 78.5 mm to (202.5, 64.8)
- moved J4 77.6 mm to (200.1, 83.7)
- moved H3 73.1 mm to (202.5, 137.7)
- moved C4 69.0 mm to (51.5, 86.1), turned to 90 degrees
- moved H1 67.0 mm to (45.5, 64.7)
- moved RV1 63.1 mm to (58.5, 91.7)
- moved H4 60.6 mm to (45.5, 137.7)
- moved J3 59.9 mm to (46.5, 75.3)
- moved C3 54.1 mm to (58.5, 88.4), turned to 0 degrees
- moved J1 52.4 mm to (73.8, 76.7), turned to 90 degrees
- moved C1 45.4 mm to (87.6, 71.4)
- moved R2 44.1 mm to (82.4, 83.5)
- moved C2 38.6 mm to (156.7, 81.0)
- moved D1 28.0 mm to (102.6, 70.2), turned to -90 degrees
- moved R1 25.8 mm to (110.2, 76.7)
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Connections:
- net MISO renamed PB1
- net MOSI renamed PB0
- J1 pad 1: Net-(J1-Pad1) -> VCC
- J2 pad 3: SCK -> PB2
- J4 pad 3: DATA -> KEYS
- RV1 pad 1: GND -> Net-(C3-Pad1)
- RV1 pad 3: Net-(C3-Pad1) -> GND
Routing:
- net GND: track 197.8 -> 522.3 mm, vias 1 -> 0
- net VCC: track 98.1 -> 294.4 mm
- net STOP0: track 0.00 -> 84.4 mm
- net SCK: track 84.3 -> 0.00 mm
- net STOP1: track 0.00 -> 73.1 mm
- net Net-(J1-Pad1): track 68.9 -> 0.00 mm
- net PB2: track 0.00 -> 68.8 mm, vias 0 -> 1
- net STOP2: track 0.00 -> 59.7 mm
- net STOP3: track 0.00 -> 55.8 mm
- net PB0: track 30.2 -> 78.6 mm
- net Net-(U2-Pad4): track 29.1 -> 75.5 mm
- net STOP4: track 0.00 -> 45.3 mm
- net STOP5: track 0.00 -> 42.1 mm
- net ~{RESET}: track 21.7 -> 60.7 mm, vias 0 -> 1
- net KEYS: track 0.00 -> 34.4 mm
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Other:
- board size 32 x 100 mm -> 164 x 80 mm
- board text added: "0"
- board text added: "1"
- board text added: "2"
- board text added: "3"
- board text added: "4"
- board text added: "5"
- board text added: "6"
- board text added: "7"
- board text added: "8"
- board text added: "MK Controller v2 - 2022-02-03 - joewing.net"
- board text removed: "MK Controller v1 - 2022-01-21 - joewing.net"
- board text removed: "Volume"

Commit message: Save
Parts:
- added J5: Pedal, Connector_PinHeader_2.54mm:PinHeader_1x02_P2.54mm_Vertical, F.Cu at (190.6, 65.1)
Connections:
- U2 pad 17: unconnected-(U2-Pad17) -> PEDAL
Routing:
- net PEDAL: track 0.00 -> 43.6 mm
- net GND: track 522.3 -> 528.3 mm
Other:
- board text added: "MK Controller v2 - 2022-02-04 - joewing.net"
- board text removed: "8"
- board text removed: "MK Controller v2 - 2022-02-03 - joewing.net"

Commit message: Boards ordered.
Parts:
- removed C10, C11, C12, C13, C14, C6, C7, C8, C9: 0.1u, Capacitor_THT:C_Disc_D3.0mm_W2.0mm_P2.50mm
- added SW1: Power, Connector_PinHeader_2.54mm:PinHeader_1x03_P2.54mm_Vertical, F.Cu at (91.3, 69.7)
- moved C3 74.7 mm to (132.9, 82.9), turned to 180 degrees
- moved R2 68.7 mm to (151.1, 82.9)
- moved C1 26.3 mm to (61.3, 71.4)
- moved C4 12.4 mm to (61.5, 78.8)
- moved C15 4.90 mm to (193.9, 83.6), turned to 90 degrees
- moved D1 4.13 mm to (98.5, 70.7)
- moved R1 3.62 mm to (113.8, 76.7)
- moved H1 2.03 mm to (47.5, 64.7)
- moved J3 2.00 mm to (48.5, 75.3)
- moved H4 1.97 mm to (47.5, 137.7)
- moved J4 0.10 mm to (200.0, 83.7)
Connections:
- J1 pad 1: VCC -> Net-(J1-Pad1)
Routing:
- net VCC: track 294.4 -> 370.6 mm
- net Net-(C3-Pad1): track 15.1 -> 84.3 mm
- net Net-(R2-Pad1): track 75.5 -> 6.43 mm
- net GND: track 528.3 -> 496.2 mm
- net Net-(J1-Pad1): track 0.00 -> 23.1 mm
- net Net-(C4-Pad1): track 7.05 -> 15.6 mm
- net Net-(D1-Pad2): track 9.27 -> 3.47 mm
- net PB2: track 68.8 -> 63.5 mm
- net STOP0: track 84.4 -> 88.6 mm
- net STOP1: track 73.1 -> 77.2 mm
- net STOP3: track 56.2 -> 60.3 mm
- net STOP2: track 59.7 -> 63.7 mm
- net STOP8: track 32.4 -> 36.1 mm
- net STOP7: track 20.8 -> 24.4 mm
- net STOP4: track 45.3 -> 48.5 mm
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Other:
- board size 164 x 80 mm -> 162 x 80 mm
